File: pcb/serial-charger.sch (KiCad schematic (older format))
At the start: 18 parts, among them IC1 CH340G, IC2 TP4056, P1 CONN_01X01, P2 USB_OTG, P3 CONN_01X05, P4 CONN_01X01, x1 xtal_osc

Commit message: disabled thermal shutoff from charger
Connections:
- wire segments 56 -> 57
Changed lines of the file:
@@
 LIBS:valves
 LIBS:netl
-LIBS:badge-cache
+LIBS:serial-charger-cache
 EELAYER 25 0
 EELAYER END
@@
 	6000 5750 5950 5750
 Wire Wire Line
-	5950 5750 5950 6050
+	5950 5650 5950 6050
 Text GLabel 7650 5950 2    60   BiDi ~ 0
 VBat
@@
 Wire Wire Line
 	2000 4100 2000 4250
+Wire Wire Line
+	6450 5650 5950 5650
+Connection ~ 5950 5750
 $EndSCHEMATC

Commit message: changed regulator and jumpers
Parts:
- removed 0R1, 0R2: 0R, netl:SMD_0603, symbol R
- removed D1: LED, netl:SMD_0603, symbol LED
- added C7: 10u, netl:SMD_0603, symbol C
- added D1: RGB_LED, netl:RGB_LED, symbol RGB_LED
- added J1, J2, J3, J4: jumper, netl:Jumper, symbol jumper
- added R3, R4: 1k, netl:SMD_0603, symbol R
- added U1: XC6206, TO_SOT_Packages_SMD:SOT-23, symbol XC6206
Connections:
- net labels added: V_MCU, V_SER, ~chrg, ~stby
- net labels removed: U_OUT
- wire segments 57 -> 72
Other:
- note added: "selector for communication voltages"
- note added: "short only one, dumbass."
- note added: "use battery to directly power mcu"
- note removed: "output voltage for powering the mcu"
- note removed: "place only one, dumbass."
- moved on the sheet: C1, C2, C3, C4, IC1, R2, x1

Commit message: changed charger
Parts:
- removed IC2: TP4056, SMD_Packages:SOIC-8-N, symbol TP4056
- removed J4: jumper, netl:Jumper, symbol jumper
- removed R1: 2k, netl:SMD_0603, symbol R
- added C?: C, symbol C
- added C?: 47uF, symbol C
- added D?: D, symbol D
- added L?: INDUCTOR, symbol INDUCTOR
- added R?: 2k, netl:SMD_0603, symbol R
- added U?: FM6316FE, netl:ESOP-8, symbol FM6316FE
Connections:
- net GND: now also C?.1, R?.2, U?.1 (GND)
- net VBat: now also L?.1, U?.5 (BAT)
- net V_USB: now also U?.4 (VCC)
- net ~chrg: now also U?.3 (CHRG)
- net ~stby: now also U?.2 (STBY)
- new net: R?.1, U?.6 (PROG)
- new net: C?.2, D?.2 (A), L?.2, U?.8 (LX)
- new net 5V: C?.1, C?.2, D?.1 (K), U?.7 (VOUT)
Other:
- note removed: "use battery to directly power mcu"
- moved on the sheet: C1, C2, C3, C4, C5, C6, C7, D1, IC1, J1, J2, J3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

Commit message: partyhat edition, with built in avr and li-ion holder
Parts:
- removed P1, P4: CONN_01X01, Connect:1pin, symbol CONN_01X01
- added P1: CONN_01X02, netl:18560, symbol CONN_01X02
- C8, C9: renamed from C?; footprint (none) -> netl:SMD_0603
- D2: renamed from D?; footprint (none) -> netl:SMD_0603
- gave numbers to parts that had none: 3
Connections:
- net 3V3: no longer D1.4
- net GND: now also P1.1 (P1)
- net VBat: now also P1.2 (P2)
- net V_USB: now also D1.4
Other:
- moved on the sheet: P3
Changed lines of the file:
@@
 $Descr A4 11693 8268
 encoding utf-8
-Sheet 1 1
+Sheet 1 2
 Title ""
 Date ""
@@
 L CONN_01X05 P3
 U 1 1 57C2DD7E
-P 3500 5700
-F 0 "P3" H 3500 5950 50  0000 C CNN
-F 1 "CONN_01X05" V 3600 5700 50  0000 C CNN
-F 2 "Pin_Headers:Pin_Header_Angled_1x05" H 3500 5700 50  0001 C CNN
-F 3 "" H 3500 5700 50  0000 C CNN
-	1    3500 5700
+P 4050 5700
+F 0 "P3" H 4050 5950 50  0000 C CNN
+F 1 "CONN_01X05" V 4150 5700 50  0000 C CNN
+F 2 "Pin_Headers:Pin_Header_Angled_1x05" H 4050 5700 50  0001 C CNN
+F 3 "" H 4050 5700 50  0000 C CNN
+	1    4050 5700
 	1    0    0    -1
 $EndComp
@@
 L GND #PWR03
 U 1 1 57C2E131
-P 3200 6100
-F 0 "#PWR03" H 3200 5850 50  0001 C CNN
-F 1 "GND" H 3200 5950 50  0000 C CNN
-F 2 "" H 3200 6100 50  0000 C CNN
-F 3 "" H 3200 6100 50  0000 C CNN
-	1    3200 6100
+P 3750 6100
+F 0 "#PWR03" H 3750 5850 50  0001 C CNN
+F 1 "GND" H 3750 5950 50  0000 C CNN
+F 2 "" H 3750 6100 50  0000 C CNN
+F 3 "" H 3750 6100 50  0000 C CNN
+	1    3750 6100
 	1    0    0    -1
 $EndComp
 Text GLabel 1600 3800 0    60   Input ~ 0
 V_MCU
-Text GLabel 3200 5600 0    60   Output ~ 0
+Text GLabel 3750 5600 0    60   Output ~ 0
 RX
-Text GLabel 3200 5700 0    60   Input ~ 0
+Text GLabel 3750 5700 0    60   Input ~ 0
 TX
 Text GLabel 1600 3550 0    60   Input ~ 0
@@
 	1450 5700 1350 5700
 Wire Wire Line
-	3300 5900 3200 5900
-Wire Wire Line
-	3200 5900 3200 6100
-Wire Wire Line
-	3200 5700 3300 5700
-Wire Wire Line
-	3300 5600 3200 5600
-Wire Wire Line
-	3200 5800 3300 5800
+	3850 5900 3750 5900
+Wire Wire Line
+	3750 5900 3750 6100
+Wire Wire Line
+	3750 5700 3850 5700
+Wire Wire Line
+	3850 5600 3750 5600
+Wire Wire Line
+	3750 5800 3850 5800
 Wire Wire Line
 	6400 6100 6400 6050
 Wire Wire Line
-	5100 5700 5200 5700
-Wire Wire Line
-	5200 5700 5400 5700
+	5100 5700 5400 5700
 Wire Wire Line
 	1450 5600 1350 5600
@@
 	6000 3300 6000 3550
 Wire Wire Line
-	4650 2500 4700 2500
-Wire Wire Line
-	4700 2500 6050 2500
+	4650 2500 6050 2500
 Wire Wire Line
 	6000 2600 6050 2600
@@
 	6050 2850 6000 2850
 Wire Wire Line
-	5750 3100 5800 3100
-Wire Wire Line
-	5800 3100 6050 3100
+	5750 3100 6050 3100
 Wire Wire Line
 	5800 3100 5800 3150
@@
 3V3
 Wire Wire Line
-	6200 5700 6400 5700
-Wire Wire Line
-	6400 5700 6500 5700
+	6200 5700 6500 5700
 Wire Wire Line
 	6400 5700 6400 5750
-Text GLabel 3200 5800 0    60   BiDi ~ 0
+Text GLabel 3750 5800 0    60   BiDi ~ 0
 V_MCU
 Wire Wire Line
-	3200 5500 3300 5500
+	3750 5500 3850 5500
 $Comp
 L xtal_osc x1
@@
 	5050 3100 5000 3100
 Wire Wire Line
-	5000 3000 5000 3100
-Wire Wire Line
-	5000 3100 5000 3150
+	5000 3000 5000 3150
 Wire Wire Line
 	5400 3450 5400 3550
 Wire Wire Line
-	5000 3450 5350 3450
-Wire Wire Line
-	5350 3450 5400 3450
-Wire Wire Line
-	5400 3450 5450 3450
-Wire Wire Line
-	5450 3450 5800 3450
+	5000 3450 5800 3450
 Connection ~ 5400 3450
 Wire Wire Line
@@
 	0    1    1    0
 $EndComp
-Text GLabel 3200 5500 0    60   Input ~ 0
+Text GLabel 3750 5500 0    60   Input ~ 0
 ~DTR
 Text GLabel 7100 2800 2    60   Output ~ 0
@@
 TX
 $Comp
-L GND #PWR08
+L GND #PWR07
 U 1 1 57DD73F7
 P 4900 5150
-F 0 "#PWR08" H 4900 4900 50  0001 C CNN
+F 0 "#PWR07" H 4900 4900 50  0001 C CNN
 F 1 "GND" H 4900 5000 50  0000 C CNN
 F 2 "" H 4900 5150 50  0000 C CNN
@@
 VBat
 $Comp
-L GND #PWR09
+L GND #PWR08
 U 1 1 57F8F41D
 P 2300 6100
-F 0 "#PWR09" H 2300 5850 50  0001 C CNN
+F 0 "#PWR08" H 2300 5850 50  0001 C CNN
 F 1 "GND" H 2300 5950 50  0000 C CNN
 F 2 "" H 2300 6100 60  0000 C CNN
@@
 $EndComp
 Wire Wire Line
-	2300 5850 2300 5950
-Wire Wire Line
-	2300 5950 2300 6100
-Wire Wire Line
-	2300 5400 2300 5500
-Wire Wire Line
-	2300 5500 2300 5550
-$Comp
-L CONN_01X01 P1
-U 1 1 57F8F79D
-P 2600 5500
-F 0 "P1" H 2600 5600 50  0000 C CNN
-F 1 "CONN_01X01" V 2700 5500 50  0000 C CNN
-F 2 "Connect:1pin" H 2600 5500 50  0001 C CNN
-F 3 "" H 2600 5500 50  0000 C CNN
-	1    2600 5500
-	1    0    0    -1
-$EndComp
-$Comp
-L CONN_01X01 P4
-U 1 1 57F8F92C
-P 2600 5950
-F 0 "P4" H 2600 6050 50  0000 C CNN
-F 1 "CONN_01X01" V 2700 5950 50  0000 C CNN
-F 2 "Connect:1pin" H 2600 5950 50  0001 C CNN
-F 3 "" H 2600 5950 50  0000 C CNN
-	1    2600 5950
-	1    0    0    -1
-$EndComp
-Wire Wire Line
-	2400 5950 2300 5950
+	2300 5850 2300 6100
+Wire Wire Line
+	2300 5400 2300 5550
+Wire Wire Line
+	2300 5950 2650 5950
 Connection ~ 2300 5950
 Wire Wire Line
-	2400 5500 2300 5500
+	2300 5500 2650 5500
 Connection ~ 2300 5500
 Wire Wire Line
-	2050 3550 2050 3800
-Wire Wire Line
-	2050 3800 2050 4050
-$Comp
-L GND #PWR010
+	2050 3550 2050 4050
+$Comp
+L GND #PWR09
 U 1 1 587A1404
 P 5800 6100
-F 0 "#PWR010" H 5800 5850 50  0001 C CNN
+F 0 "#PWR09" H 5800 5850 50  0001 C CNN
 F 1 "GND" H 5800 5950 50  0000 C CNN
 F 2 "" H 5800 6100 50  0000 C CNN
@@
 	1600 3550 1650 3550
 Wire Wire Line
-	1950 3800 2050 3800
-Wire Wire Line
-	2050 3800 2150 3800
+	1950 3800 2150 3800
 Connection ~ 2050 3800
 Wire Wire Line
@@
 $EndComp
 $Comp
-L GND #PWR011
+L GND #PWR010
 U 1 1 589F9E27
 P 4700 3550
-F 0 "#PWR011" H 4700 3300 50  0001 C CNN
+F 0 "#PWR010" H 4700 3300 50  0001 C CNN
 F 1 "GND" H 4700 3400 50  0000 C CNN
 F 2 "" H 4700 3550 50  0000 C CNN
@@
 $EndComp
 Text GLabel 1200 4750 0    60   Input ~ 0
-3V3
+V_USB
 Wire Wire Line
 	1250 4750 1200 4750
@@
 	2250 4600 2200 4600
 $Comp
-L FM6316FE U?
+L FM6316FE U2
 U 1 1 58B85FE3
 P 5800 4400
-F 0 "U?" H 5800 4700 60  0000 C CNN
+F 0 "U2" H 5800 4700 60  0000 C CNN
 F 1 "FM6316FE" H 5800 4600 60  0000 C CNN
 F 2 "netl:ESOP-8" H 5800 4100 60  0000 C CNN
@@
 5V
 Wire Wire Line
-	4700 4300 4900 4300
-Wire Wire Line
-	4900 4300 5350 4300
+	4700 4300 5350 4300
 Text GLabel 5300 4500 0    60   Output ~ 0
 ~stby
@@
 	5350 4500 5300 4500
 $Comp
-L GND #PWR?
+L GND #PWR011
 U 1 1 58B86D8C
 P 5300 5150
-F 0 "#PWR?" H 5300 4900 50  0001 C CNN
+F 0 "#PWR011" H 5300 4900 50  0001 C CNN
 F 1 "GND" H 5300 5000 50  0000 C CNN
 F 2 "" H 5300 5150 50  0000 C CNN
@@
 	5300 4600 5350 4600
 $Comp
-L R R?
+L R R1
 U 1 1 58B86F80
 P 6350 4900
-F 0 "R?" V 6430 4900 50  0000 C CNN
+F 0 "R1" V 6430 4900 50  0000 C CNN
 F 1 "2k" V 6350 4900 50  0000 C CNN
 F 2 "netl:SMD_0603" V 6280 4900 50  0001 C CNN
@@
 	5300 4600 5300 5150
 $Comp
-L GND #PWR?
+L GND #PWR012
 U 1 1 58B872A6
 P 6350 5150
-F 0 "#PWR?" H 6350 4900 50  0001 C CNN
+F 0 "#PWR012" H 6350 4900 50  0001 C CNN
 F 1 "GND" H 6350 5000 50  0000 C CNN
 F 2 "" H 6350 5150 50  0000 C CNN
@@
 $EndComp
 $Comp
-L INDUCTOR L?
+L INDUCTOR L1
 U 1 1 58B8750F
 P 6650 4300
-F 0 "L?" V 6600 4300 50  0000 C CNN
+F 0 "L1" V 6600 4300 50  0000 C CNN
 F 1 "INDUCTOR" V 6750 4300 50  0000 C CNN
-F 2 "" H 6650 4300 50  0000 C CNN
+F 2 "" H 6650 4300 50  0001 C CNN
 F 3 "" H 6650 4300 50  0000 C CNN
 	1    6650 4300
@@
 $EndComp
 $Comp
-L D D?
+L D D2
 U 1 1 58B87669
 P 6950 4600
-F 0 "D?" V 6850 4500 50  0000 C CNN
+F 0 "D2" V 6850 4500 50  0000 C CNN
 F 1 "D" V 7050 4500 50  0000 C CNN
-F 2 "" H 6950 4600 50  0000 C CNN
+F 2 "netl:SMD_0603" H 6950 4600 50  0001 C CNN
 F 3 "" H 6950 4600 50  0000 C CNN
 	1    6950 4600
@@
 $EndComp
 $Comp
-L C C?
+L C C8
 U 1 1 58B8771C
 P 6700 4600
-F 0 "C?" H 6550 4700 50  0000 L CNN
+F 0 "C8" H 6550 4700 50  0000 L CNN
 F 1 "C" H 6600 4500 50  0000 L CNN
-F 2 "" H 6738 4450 50  0000 C CNN
+F 2 "netl:SMD_0603" H 6738 4450 50  0001 C CNN
 F 3 "" H 6700 4600 50  0000 C CNN
 	1    6700 4600
@@
 $EndComp
 Wire Wire Line
-	6250 4400 6700 4400
-Wire Wire Line
-	6700 4400 6950 4400
+	6250 4400 6950 4400
 Wire Wire Line
 	6700 4400 6700 4450
 Wire Wire Line
-	6950 4300 6950 4400
-Wire Wire Line
-	6950 4400 6950 4450
+	6950 4300 6950 4450
 Connection ~ 6700 4400
 Wire Wire Line
-	6250 4300 6300 4300
-Wire Wire Line
-	6300 4300 6350 4300
+	6250 4300 6350 4300
 Connection ~ 6950 4400
 Wire Wire Line
@@
 	6550 4500 6550 4750
 Wire Wire Line
-	6550 4750 6700 4750
-Wire Wire Line
-	6700 4750 6950 4750
-Wire Wire Line
-	6950 4750 7150 4750
+	6550 4750 7150 4750
 Connection ~ 6700 4750
 Connection ~ 6950 4750
 $Comp
-L C C?
+L C C9
 U 1 1 58B8A12B
 P 6700 4950
-F 0 "C?" H 6550 5050 50  0000 L CNN
+F 0 "C9" H 6550 5050 50  0000 L CNN
 F 1 "47uF" H 6500 4850 50  0000 L CNN
-F 2 "" H 6738 4800 50  0000 C CNN
+F 2 "netl:SMD_0603" H 6738 4800 50  0001 C CNN
 F 3 "" H 6700 4950 50  0000 C CNN
 	1    6700 4950
@@
 	6350 5050 6350 5150
 $Comp
-L GND #PWR?
+L GND #PWR013
 U 1 1 58B8A61A
 P 6700 5150
-F 0 "#PWR?" H 6700 4900 50  0001 C CNN
+F 0 "#PWR013" H 6700 4900 50  0001 C CNN
 F 1 "GND" H 6700 5000 50  0000 C CNN
 F 2 "" H 6700 5150 50  0000 C CNN
@@
 	4700 2850 4700 2500
 Connection ~ 4700 2500
+$Sheet
+S 9100 3800 1600 1500
+U 58B9D13D
+F0 "avr" 60
+F1 "avr.sch" 60
+F2 "gnd" I L 9100 5200 60
+F3 "VCC" I L 9100 3900 60
+F4 "~DTR" I L 9100 4600 60
+F5 "RX" I L 9100 4700 60
+F6 "TX" O L 9100 4800 60
+$EndSheet
+$Comp
+L GND #PWR014
+U 1 1 58B9EA67
+P 9000 5250
+F 0 "#PWR014" H 9000 5000 50  0001 C CNN
+F 1 "GND" H 9000 5100 50  0000 C CNN
+F 2 "" H 9000 5250 50  0000 C CNN
+F 3 "" H 9000 5250 50  0000 C CNN
+	1    9000 5250
+	1    0    0    -1
+$EndComp
+Text GLabel 9000 3900 0    60   Input ~ 0
+5V
+Wire Wire Line
+	9000 3900 9100 3900
+Wire Wire Line
+	9100 5200 9000 5200
+Wire Wire Line
+	9000 5200 9000 5250
+Text GLabel 9050 4700 0    60   Input ~ 0
+TX
+Text GLabel 9050 4800 0    60   Output ~ 0
+RX
+Text GLabel 9050 4600 0    60   Input ~ 0
+~DTR
+Wire Wire Line
+	9050 4600 9100 4600
+Wire Wire Line
+	9100 4700 9050 4700
+Wire Wire Line
+	9050 4800 9100 4800
+$Comp
+L CONN_01X02 P1
+U 1 1 58BA30E4
+P 2850 5750
+F 0 "P1" H 2850 5900 50  0000 C CNN
+F 1 "CONN_01X02" V 2950 5750 50  0000 C CNN
+F 2 "netl:18560" H 2850 6050 50  0000 C CNN
+F 3 "" H 2850 5750 50  0000 C CNN
+	1    2850 5750
+	1    0    0    1
+$EndComp
+Wire Wire Line
+	2650 5500 2650 5700
+Wire Wire Line
+	2650 5950 2650 5800
 $EndSCHEMATC

Commit message: layout mostly done
Parts:
- removed J2: jumper, netl:Jumper, symbol jumper
- removed P3: CONN_01X05, Pin_Headers:Pin_Header_Angled_1x05, symbol CONN_01X05
- added P3: CONN_01X04, Socket_Strips:Socket_Strip_Angled_1x04, symbol CONN_01X04
- L1: footprint (none) -> netl:7x7_Inductor
- renumbered J3 to J2
Connections:
- net 5V: now also P3.4 (P4)
- net GND: now also P3.1 (P1)
- net RX: now also P3.3 (P3)
- net TX: now also P3.2 (P2)
Other:
- moved on the sheet: J2
Changed lines of the file:
@@
 	1    0    0    -1
 $EndComp
-$Comp
-L CONN_01X05 P3
-U 1 1 57C2DD7E
-P 4050 5700
-F 0 "P3" H 4050 5950 50  0000 C CNN
-F 1 "CONN_01X05" V 4150 5700 50  0000 C CNN
-F 2 "Pin_Headers:Pin_Header_Angled_1x05" H 4050 5700 50  0001 C CNN
-F 3 "" H 4050 5700 50  0000 C CNN
-	1    4050 5700
-	1    0    0    -1
-$EndComp
-$Comp
-L GND #PWR03
-U 1 1 57C2E131
-P 3750 6100
-F 0 "#PWR03" H 3750 5850 50  0001 C CNN
-F 1 "GND" H 3750 5950 50  0000 C CNN
-F 2 "" H 3750 6100 50  0000 C CNN
-F 3 "" H 3750 6100 50  0000 C CNN
-	1    3750 6100
-	1    0    0    -1
-$EndComp
-Text GLabel 1600 3800 0    60   Input ~ 0
-V_MCU
-Text GLabel 3750 5600 0    60   Output ~ 0
-RX
-Text GLabel 3750 5700 0    60   Input ~ 0
-TX
 Text GLabel 1600 3550 0    60   Input ~ 0
 V_USB
@@
 selector for communication voltages
 $Comp
-L GND #PWR04
+L GND #PWR03
 U 1 1 57C325B8
 P 6400 6100
-F 0 "#PWR04" H 6400 5850 50  0001 C CNN
+F 0 "#PWR03" H 6400 5850 50  0001 C CNN
 F 1 "GND" H 6400 5950 50  0000 C CNN
 F 2 "" H 6400 6100 50  0000 C CNN
@@
 $EndComp
 $Comp
-L GND #PWR05
+L GND #PWR04
 U 1 1 57C5D0E9
 P 6000 3550
-F 0 "#PWR05" H 6000 3300 50  0001 C CNN
+F 0 "#PWR04" H 6000 3300 50  0001 C CNN
 F 1 "GND" H 6000 3400 50  0000 C CNN
 F 2 "" H 6000 3550 50  0000 C CNN
@@
 D+
 $Comp
-L GND #PWR06
+L GND #PWR05
 U 1 1 57C5EAC0
 P 5400 3550
-F 0 "#PWR06" H 5400 3300 50  0001 C CNN
+F 0 "#PWR05" H 5400 3300 50  0001 C CNN
 F 1 "GND" H 5400 3400 50  0000 C CNN
 F 2 "" H 5400 3550 50  0000 C CNN
@@
 Wire Wire Line
 	1450 5700 1350 5700
-Wire Wire Line
-	3850 5900 3750 5900
-Wire Wire Line
-	3750 5900 3750 6100
-Wire Wire Line
-	3750 5700 3850 5700
-Wire Wire Line
-	3850 5600 3750 5600
-Wire Wire Line
-	3750 5800 3850 5800
 Wire Wire Line
 	6400 6100 6400 6050
@@
 Wire Wire Line
 	6400 5700 6400 5750
-Text GLabel 3750 5800 0    60   BiDi ~ 0
-V_MCU
-Wire Wire Line
-	3750 5500 3850 5500
 $Comp
 L xtal_osc x1
@@
 	0    1    1    0
 $EndComp
-Text GLabel 3750 5500 0    60   Input ~ 0
-~DTR
 Text GLabel 7100 2800 2    60   Output ~ 0
 ~DTR
@@
 TX
 $Comp
-L GND #PWR07
+L GND #PWR06
 U 1 1 57DD73F7
 P 4900 5150
-F 0 "#PWR07" H 4900 4900 50  0001 C CNN
+F 0 "#PWR06" H 4900 4900 50  0001 C CNN
 F 1 "GND" H 4900 5000 50  0000 C CNN
 F 2 "" H 4900 5150 50  0000 C CNN
@@
 VBat
 $Comp
-L GND #PWR08
+L GND #PWR07
 U 1 1 57F8F41D
 P 2300 6100
-F 0 "#PWR08" H 2300 5850 50  0001 C CNN
+F 0 "#PWR07" H 2300 5850 50  0001 C CNN
 F 1 "GND" H 2300 5950 50  0000 C CNN
 F 2 "" H 2300 6100 60  0000 C CNN
@@
 	2300 5500 2650 5500
 Connection ~ 2300 5500
-Wire Wire Line
-	2050 3550 2050 4050
-$Comp
-L GND #PWR09
+$Comp
+L GND #PWR08
 U 1 1 587A1404
 P 5800 6100
-F 0 "#PWR09" H 5800 5850 50  0001 C CNN
+F 0 "#PWR08" H 5800 5850 50  0001 C CNN
 F 1 "GND" H 5800 5950 50  0000 C CNN
 F 2 "" H 5800 6100 50  0000 C CNN
@@
 	1    0    0    -1
 $EndComp
+Text GLabel 2150 3800 2    60   Output ~ 0
+V_SER
+Text GLabel 1600 3800 0    60   Input ~ 0
+3V3
 $Comp
 L jumper J2
-U 1 1 589F4D0E
+U 1 1 589F5A87
 P 1800 3800
 F 0 "J2" H 1800 3700 60  0000 C CNN
@@
 	1    0    0    -1
 $EndComp
-Text GLabel 2150 3800 2    60   Output ~ 0
-V_SER
-Text GLabel 1600 4050 0    60   Input ~ 0
-3V3
-$Comp
-L jumper J3
-U 1 1 589F5A87
-P 1800 4050
-F 0 "J3" H 1800 3950 60  0000 C CNN
-F 1 "jumper" H 1800 4150 60  0000 C CNN
-F 2 "netl:Jumper" H 1800 4050 60  0001 C CNN
-F 3 "" H 1800 4050 60  0000 C CNN
-	1    1800 4050
-	1    0    0    -1
-$EndComp
-Wire Wire Line
-	1600 4050 1650 4050
-Wire Wire Line
-	2050 4050 1950 4050
+Wire Wire Line
+	1600 3800 1650 3800
 Wire Wire Line
 	2050 3550 1950 3550
 Wire Wire Line
 	1600 3550 1650 3550
-Wire Wire Line
-	1950 3800 2150 3800
-Connection ~ 2050 3800
-Wire Wire Line
-	1650 3800 1600 3800
 $Comp
 L C C7
@@
 $EndComp
 $Comp
-L GND #PWR010
+L GND #PWR09
 U 1 1 589F9E27
 P 4700 3550
-F 0 "#PWR010" H 4700 3300 50  0001 C CNN
+F 0 "#PWR09" H 4700 3300 50  0001 C CNN
 F 1 "GND" H 4700 3400 50  0000 C CNN
 F 2 "" H 4700 3550 50  0000 C CNN
@@
 	5350 4500 5300 4500
 $Comp
-L GND #PWR011
+L GND #PWR010
 U 1 1 58B86D8C
 P 5300 5150
-F 0 "#PWR011" H 5300 4900 50  0001 C CNN
+F 0 "#PWR010" H 5300 4900 50  0001 C CNN
 F 1 "GND" H 5300 5000 50  0000 C CNN
 F 2 "" H 5300 5150 50  0000 C CNN
@@
 	5300 4600 5300 5150
 $Comp
-L GND #PWR012
+L GND #PWR011
 U 1 1 58B872A6
 P 6350 5150
-F 0 "#PWR012" H 6350 4900 50  0001 C CNN
+F 0 "#PWR011" H 6350 4900 50  0001 C CNN
 F 1 "GND" H 6350 5000 50  0000 C CNN
 F 2 "" H 6350 5150 50  0000 C CNN
@@
 F 0 "L1" V 6600 4300 50  0000 C CNN
 F 1 "INDUCTOR" V 6750 4300 50  0000 C CNN
-F 2 "" H 6650 4300 50  0001 C CNN
+F 2 "netl:7x7_Inductor" H 6650 4300 50  0001 C CNN
 F 3 "" H 6650 4300 50  0000 C CNN
 	1    6650 4300
@@
 	6350 5050 6350 5150
 $Comp
-L GND #PWR013
+L GND #PWR012
 U 1 1 58B8A61A
 P 6700 5150
-F 0 "#PWR013" H 6700 4900 50  0001 C CNN
+F 0 "#PWR012" H 6700 4900 50  0001 C CNN
 F 1 "GND" H 6700 5000 50  0000 C CNN
 F 2 "" H 6700 5150 50  0000 C CNN
@@
 $EndSheet
 $Comp
-L GND #PWR014
+L GND #PWR013
 U 1 1 58B9EA67
 P 9000 5250
-F 0 "#PWR014" H 9000 5000 50  0001 C CNN
+F 0 "#PWR013" H 9000 5000 50  0001 C CNN
 F 1 "GND" H 9000 5100 50  0000 C CNN
 F 2 "" H 9000 5250 50  0000 C CNN
@@
 Wire Wire Line
 	2650 5950 2650 5800
+$Comp
+L CONN_01X04 P3
+U 1 1 58BAC680
+P 3750 5850
+F 0 "P3" H 3750 6100 50  0000 C CNN
+F 1 "CONN_01X04" V 3850 5850 50  0000 C CNN
+F 2 "Socket_Strips:Socket_Strip_Angled_1x04" H 3750 5850 50  0000 C CNN
+F 3 "" H 3750 5850 50  0000 C CNN
+	1    3750 5850
+	1    0    0    1
+$EndComp
+Text GLabel 3500 5800 0    60   Output ~ 0
+RX
+Text GLabel 3500 5900 0    60   Input ~ 0
+TX
+$Comp
+L GND #PWR014
+U 1 1 58BACB26
+P 3500 6000
+F 0 "#PWR014" H 3500 5750 50  0001 C CNN
+F 1 "GND" H 3500 5850 50  0000 C CNN
+F 2 "" H 3500 6000 50  0000 C CNN
+F 3 "" H 3500 6000 50  0000 C CNN
+	1    3500 6000
+	1    0    0    -1
+$EndComp
+Text GLabel 3500 5700 0    60   Input ~ 0
+5V
+Wire Wire Line
+	3500 5700 3550 5700
+Wire Wire Line
+	3550 5800 3500 5800
+Wire Wire Line
+	3500 5900 3550 5900
+Wire Wire Line
+	3550 6000 3500 6000
+Wire Wire Line
+	1950 3800 2150 3800
+Connection ~ 2050 3800
+Wire Wire Line
+	2050 3800 2050 3550
 $EndSCHEMATC

Commit message: first prototype
Parts:
- P3: footprint Socket_Strips:Socket_Strip_Angled_1x04 -> netl:JST-2mm_4Pin
Changed lines of the file:
@@
 F 0 "P3" H 3750 6100 50  0000 C CNN
 F 1 "CONN_01X04" V 3850 5850 50  0000 C CNN
-F 2 "Socket_Strips:Socket_Strip_Angled_1x04" H 3750 5850 50  0000 C CNN
+F 2 "netl:JST-2mm_4Pin" H 3750 6250 50  0000 C CNN
 F 3 "" H 3750 5850 50  0000 C CNN
 	1    3750 5850
