File: pcb/_saved_serial-charger.sch (KiCad schematic (older format))
At the start: 12 parts, among them J101 jumper, J102 jumper, P101 USB_OTG, P102 CONN_01X02, P103 CONN_01X04, U101 XC6206

Commit message: changed LED and boost converters Diode footprints. renumbered components
Parts:
- R101, R102, R103: value 1k -> 4.7k
Changed lines of the file:
@@
 $EndComp
 $Comp
-L GND #PWR101
+L GND #PWR01
 U 1 1 55AEBF75
 P 2200 3300
-F 0 "#PWR101" H 2200 3050 50  0001 C CNN
+F 0 "#PWR01" H 2200 3050 50  0001 C CNN
 F 1 "GND" H 2200 3150 50  0000 C CNN
 F 2 "" H 2200 3300 60  0000 C CNN
@@
 $EndComp
 $Comp
-L GND #PWR104
+L GND #PWR02
 U 1 1 579ECB3C
 P 6550 3500
-F 0 "#PWR104" H 6550 3250 50  0001 C CNN
+F 0 "#PWR02" H 6550 3250 50  0001 C CNN
 F 1 "GND" H 6550 3350 50  0000 C CNN
 F 2 "" H 6550 3500 50  0000 C CNN
@@
 selector for communication voltages
 $Comp
-L GND #PWR106
+L GND #PWR03
 U 1 1 57C325B8
 P 7750 3500
-F 0 "#PWR106" H 7750 3250 50  0001 C CNN
+F 0 "#PWR03" H 7750 3250 50  0001 C CNN
 F 1 "GND" H 7750 3350 50  0000 C CNN
 F 2 "" H 7750 3500 50  0000 C CNN
@@
 P 7350 2200
 F 0 "R103" V 7430 2200 50  0000 C CNN
-F 1 "1k" V 7350 2200 50  0000 C CNN
+F 1 "4.7k" V 7350 2200 50  0000 C CNN
 F 2 "netl:SMD_0603" V 7280 2200 50  0001 C CNN
 F 3 "" H 7350 2200 50  0000 C CNN
@@
 $EndComp
 $Comp
-L GND #PWR102
+L GND #PWR04
 U 1 1 57F8F41D
 P 5200 3300
-F 0 "#PWR102" H 5200 3050 50  0001 C CNN
+F 0 "#PWR04" H 5200 3050 50  0001 C CNN
 F 1 "GND" H 5200 3150 50  0000 C CNN
 F 2 "" H 5200 3300 60  0000 C CNN
@@
 $EndComp
 $Comp
-L GND #PWR105
+L GND #PWR05
 U 1 1 587A1404
 P 7150 3500
-F 0 "#PWR105" H 7150 3250 50  0001 C CNN
+F 0 "#PWR05" H 7150 3250 50  0001 C CNN
 F 1 "GND" H 7150 3350 50  0000 C CNN
 F 2 "" H 7150 3500 50  0000 C CNN
@@
 P 7350 2050
 F 0 "R102" V 7430 2050 50  0000 C CNN
-F 1 "1k" V 7350 2050 50  0000 C CNN
+F 1 "4.7k" V 7350 2050 50  0000 C CNN
 F 2 "netl:SMD_0603" V 7280 2050 50  0001 C CNN
 F 3 "" H 7350 2050 50  0000 C CNN
@@
 P 7350 1900
 F 0 "R101" V 7430 1900 50  0000 C CNN
-F 1 "1k" V 7350 1900 50  0000 C CNN
+F 1 "4.7k" V 7350 1900 50  0000 C CNN
 F 2 "netl:SMD_0603" V 7280 1900 50  0001 C CNN
 F 3 "" H 7350 1900 50  0000 C CNN
@@
 $EndSheet
 $Comp
-L GND #PWR107
+L GND #PWR06
 U 1 1 58B9EA67
 P 7900 5500
-F 0 "#PWR107" H 7900 5250 50  0001 C CNN
+F 0 "#PWR06" H 7900 5250 50  0001 C CNN
 F 1 "GND" H 7900 5350 50  0000 C CNN
 F 2 "" H 7900 5500 50  0000 C CNN
@@
 	5850 4950 5850 4550
 $Comp
-L GND #PWR103
+L GND #PWR07
 U 1 1 58BACB26
 P 5950 4700
-F 0 "#PWR103" H 5950 4450 50  0001 C CNN
+F 0 "#PWR07" H 5950 4450 50  0001 C CNN
 F 1 "GND" H 5950 4550 50  0000 C CNN
 F 2 "" H 5950 4700 50  0000 C CNN
