File: pcb/FM6316FE.sch (KiCad schematic (older format))
At the start: 8 parts

Commit message: changed LED and boost converters Diode footprints. renumbered components
Parts:
- gave numbers to parts that had none: 8
Connections:
- wire segments 32 -> 24
Changed lines of the file:
@@
 $EndDescr
 $Comp
-L GND #PWR?
+L GND #PWR301
 U 1 1 58D7F4CB
 P 4800 4200
-F 0 "#PWR?" H 4800 3950 50  0001 C CNN
+F 0 "#PWR301" H 4800 3950 50  0001 C CNN
 F 1 "GND" H 4800 4050 50  0000 C CNN
 F 2 "" H 4800 4200 50  0000 C CNN
@@
 $EndComp
 $Comp
-L C C?
+L C C301
 U 1 1 58D7F4D1
 P 4800 3800
-F 0 "C?" H 4825 3900 50  0000 L CNN
+F 0 "C301" H 4825 3900 50  0000 L CNN
 F 1 "10u" H 4825 3700 50  0000 L CNN
 F 2 "netl:SMD_0603" H 4838 3650 50  0001 C CNN
@@
 $EndComp
 $Comp
-L FM6316FE U?
+L FM6316FE U301
 U 1 1 58D7F4DA
 P 5700 3450
-F 0 "U?" H 5700 3750 60  0000 C CNN
+F 0 "U301" H 5700 3750 60  0000 C CNN
 F 1 "FM6316FE" H 5700 3650 60  0000 C CNN
 F 2 "netl:ESOP-8" H 5700 3150 60  0000 C CNN
@@
 $EndComp
 $Comp
-L GND #PWR?
+L GND #PWR302
 U 1 1 58D7F4E8
 P 5200 4200
-F 0 "#PWR?" H 5200 3950 50  0001 C CNN
+F 0 "#PWR302" H 5200 3950 50  0001 C CNN
 F 1 "GND" H 5200 4050 50  0000 C CNN
 F 2 "" H 5200 4200 50  0000 C CNN
@@
 $EndComp
 $Comp
-L R R?
+L R R301
 U 1 1 58D7F4EF
 P 6200 3950
-F 0 "R?" H 6300 4050 50  0000 C CNN
+F 0 "R301" H 6300 4050 50  0000 C CNN
 F 1 "2k" V 6200 3950 50  0000 C CNN
 F 2 "netl:SMD_0603" V 6130 3950 50  0001 C CNN
@@
 $EndComp
 $Comp
-L GND #PWR?
+L GND #PWR303
 U 1 1 58D7F4F7
 P 6200 4200
-F 0 "#PWR?" H 6200 3950 50  0001 C CNN
+F 0 "#PWR303" H 6200 3950 50  0001 C CNN
 F 1 "GND" H 6200 4050 50  0000 C CNN
 F 2 "" H 6200 4200 50  0000 C CNN
@@
 $EndComp
 $Comp
-L D D?
+L D D301
 U 1 1 58D7F504
 P 7400 3350
-F 0 "D?" V 7300 3250 50  0000 C CNN
+F 0 "D301" V 7300 3250 50  0000 C CNN
 F 1 "D" V 7500 3250 50  0000 C CNN
 F 2 "netl:DO-214AC" H 7400 3350 50  0001 C CNN
@@
 $EndComp
 $Comp
-L C C?
+L C C303
 U 1 1 58D7F50B
 P 7400 3600
-F 0 "C?" V 7300 3650 50  0000 L CNN
+F 0 "C303" V 7300 3650 50  0000 L CNN
 F 1 "2nF" V 7500 3650 50  0000 L CNN
 F 2 "netl:SMD_0603" H 7438 3450 50  0001 C CNN
@@
 $EndComp
 $Comp
-L GND #PWR?
+L GND #PWR305
 U 1 1 58D7F528
 P 7650 4200
-F 0 "#PWR?" H 7650 3950 50  0001 C CNN
+F 0 "#PWR305" H 7650 3950 50  0001 C CNN
 F 1 "GND" H 7650 4050 50  0000 C CNN
 F 2 "" H 7650 4200 50  0000 C CNN
@@
 5V_OUT
 $Comp
-L C C?
+L C C302
 U 1 1 58D83030
 P 6450 3950
-F 0 "C?" H 6500 4050 50  0000 L CNN
+F 0 "C302" H 6500 4050 50  0000 L CNN
 F 1 "10uF" H 6500 3850 50  0000 L CNN
 F 2 "netl:SMD_0603" H 6488 3800 50  0001 C CNN
@@
 	4800 3950 4800 4200
 Wire Wire Line
-	4600 3350 4800 3350
-Wire Wire Line
-	4800 3350 5250 3350
+	4600 3350 5250 3350
 Wire Wire Line
 	5250 3450 5200 3450
@@
 	7650 4100 7650 4200
 $Comp
-L INDUCTOR L?
+L INDUCTOR L301
 U 1 1 58D7F4FD
 P 6800 3350
-F 0 "L?" V 6750 3350 50  0000 C CNN
+F 0 "L301" V 6750 3350 50  0000 C CNN
 F 1 "3.3uH" V 6900 3350 50  0000 C CNN
 F 2 "netl:7x7_Inductor" H 6800 3350 50  0001 C CNN
@@
 	7150 3600 7250 3600
 Wire Wire Line
-	7100 3350 7150 3350
-Wire Wire Line
-	7150 3350 7250 3350
+	7100 3350 7250 3350
 Connection ~ 7150 3350
 Wire Wire Line
-	7550 3350 7650 3350
-Wire Wire Line
-	7650 3350 7750 3350
-$Comp
-L GND #PWR?
+	7550 3350 7750 3350
+$Comp
+L GND #PWR304
 U 1 1 58D86C8C
 P 6450 4200
-F 0 "#PWR?" H 6450 3950 50  0001 C CNN
+F 0 "#PWR304" H 6450 3950 50  0001 C CNN
 F 1 "GND" H 6450 4050 50  0000 C CNN
 F 2 "" H 6450 4200 50  0000 C CNN
@@
 	6450 4100 6450 4200
 Wire Wire Line
-	6450 3250 6450 3350
-Wire Wire Line
-	6450 3350 6450 3800
-Wire Wire Line
-	7150 3350 7150 3450
-Wire Wire Line
-	7150 3450 7150 3600
-Wire Wire Line
-	6150 3350 6450 3350
-Wire Wire Line
-	6450 3350 6500 3350
+	6450 3250 6450 3800
+Wire Wire Line
+	7150 3350 7150 3600
+Wire Wire Line
+	6150 3350 6500 3350
 Wire Wire Line
 	6150 3450 7150 3450
@@
 	7050 3550 6150 3550
 Wire Wire Line
-	7650 3800 7650 3750
-Wire Wire Line
-	7650 3750 7650 3600
-Wire Wire Line
-	7650 3600 7650 3350
+	7650 3350 7650 3800
 Connection ~ 7650 3350
 Wire Wire Line
@@
 Connection ~ 7650 3600
 $Comp
-L C C?
+L C C304
 U 1 1 58D7F51D
 P 7650 3950
-F 0 "C?" H 7700 4050 50  0000 L CNN
+F 0 "C304" H 7700 4050 50  0000 L CNN
 F 1 "47uF" H 7700 3850 50  0000 L CNN
 F 2 "netl:SMD_0603" H 7688 3800 50  0001 C CNN

Commit message: cleaned up component values, rebuilt BOM
Parts:
- C302: value 10uF -> 10u
- C303: value 2nF -> 2n
- C304: value 47uF -> 47u
- D301: value D -> 1N5822
- L301: value 3.3uH -> 3.3u
Changed lines of the file:
@@
 P 7400 3350
 F 0 "D301" V 7300 3250 50  0000 C CNN
-F 1 "D" V 7500 3250 50  0000 C CNN
+F 1 "1N5822" V 7500 3250 50  0000 C CNN
 F 2 "netl:DO-214AC" H 7400 3350 50  0001 C CNN
 F 3 "" H 7400 3350 50  0000 C CNN
@@
 P 7400 3600
 F 0 "C303" V 7300 3650 50  0000 L CNN
-F 1 "2nF" V 7500 3650 50  0000 L CNN
+F 1 "2n" V 7500 3650 50  0000 L CNN
 F 2 "netl:SMD_0603" H 7438 3450 50  0001 C CNN
 F 3 "" H 7400 3600 50  0000 C CNN
@@
 P 6450 3950
 F 0 "C302" H 6500 4050 50  0000 L CNN
-F 1 "10uF" H 6500 3850 50  0000 L CNN
+F 1 "10u" H 6500 3850 50  0000 L CNN
 F 2 "netl:SMD_0603" H 6488 3800 50  0001 C CNN
 F 3 "" H 6450 3950 50  0000 C CNN
@@
 P 6800 3350
 F 0 "L301" V 6750 3350 50  0000 C CNN
-F 1 "3.3uH" V 6900 3350 50  0000 C CNN
+F 1 "3.3u" V 6900 3350 50  0000 C CNN
 F 2 "netl:7x7_Inductor" H 6800 3350 50  0001 C CNN
 F 3 "" H 6800 3350 50  0000 C CNN
@@
 P 7650 3950
 F 0 "C304" H 7700 4050 50  0000 L CNN
-F 1 "47uF" H 7700 3850 50  0000 L CNN
+F 1 "47u" H 7700 3850 50  0000 L CNN
 F 2 "netl:SMD_0603" H 7688 3800 50  0001 C CNN
 F 3 "" H 7650 3950 50  0000 C CNN

Commit message: reworked bms and mcu to use seeed components
Parts:
- removed C301, C302: 10u, netl:SMD_0603, symbol C
- removed C303: 2n, netl:SMD_0603, symbol C
- removed C304: 47u, netl:SMD_0603, symbol C
- removed D301: 1N5822, netl:DO-214AC, symbol D
- removed L301: 3.3u, netl:7x7_Inductor, symbol INDUCTOR
- removed R301: 2k, netl:SMD_0603, symbol R
- removed U301: FM6316FE, netl:ESOP-8, symbol FM6316FE
- added C301, C302: CERAMIC-4.7UF-10V-10%-X5R_0603_, SeeedOPL-Capacitor-2016:C0603, symbol CERAMIC-4.7UF-10V-10%-X5R_0603_
- added C303: CERAMIC-4.7NF-50V-10%-X7R_0603_, SeeedOPL-Capacitor-2016:C0603, symbol CERAMIC-4.7NF-50V-10%-X7R_0603_
- added C304: CERAMIC-33NF-50V-10%-X7R_0603_, SeeedOPL-Capacitor-2016:C0603, symbol CERAMIC-33NF-50V-10%-X7R_0603_
- added C305: CERAMIC-100NF-50V-10%-X7R_0603_, SeeedOPL-Capacitor-2016:C0603, symbol CERAMIC-100NF-50V-10%-X7R_0603_
- added C306, C307: CERAMIC-22UF-6.3V-20%-X5R_0805_, SeeedOPL-Capacitor-2016:C0805, symbol CERAMIC-22UF-6.3V-20%-X5R_0805_
- added D301, D302: SMD-DIODE-SCHOTTKY-28V-5A_DO-214AA_, SeeedOPL-Diode-2016:DO-214AA, symbol SMD-DIODE-SCHOTTKY-28V-5A_DO-214AA_
- added L301: SMD-INDUCTOR-10UH-20%_2P-6X6MM_, SeeedOPL-Inductor-2016:SMD-2P-L6.0XW6.0XH3.0MM, symbol SMD-INDUCTOR-10UH-20%_2P-6X6MM_
- added R301, R308: SMD-RES-10K-1%-1_10W_0603_, SeeedOPL-Resistor-2016:R0603, symbol SMD-RES-10K-1%-1_10W_0603_
- added R302: SMD-RES-0R-5%-1_10W_0603_, SeeedOPL-Resistor-2016:R0603, symbol SMD-RES-0R-5%-1_10W_0603_
- added R303: SMD-RES-3.6R-5%-1_10W_0603_, SeeedOPL-Resistor-2016:R0603, symbol SMD-RES-3.6R-5%-1_10W_0603_
- added R304: SMD-RES-0R-5%-1_10W_0603_, Resistors_SMD:R_0603, symbol SMD-RES-0R-5%-1_10W_0603_
- added R305: SMD-RES-10K-5%-1_10W_0603_, SeeedOPL-Resistor-2016:R0603, symbol SMD-RES-10K-5%-1_10W_0603_
- added R306: SMD-RES-3.9K-5%-1_10W_0603_, SeeedOPL-Resistor-2016:R0603, symbol SMD-RES-3.9K-5%-1_10W_0603_
- added R307: SMD-RES-30K-1%-1_10W_0603_, SeeedOPL-Resistor-2016:R0603, symbol SMD-RES-30K-1%-1_10W_0603_
- added U301: PMIC-CN3065_DFN8_, SeeedOPL-IC-2016:DFN8G-0.5-3X3MM, symbol PMIC-CN3065_DFN8_
- added U302: PMIC-ISL97516IUZ-TK_MSOP8_, SeeedOPL-IC-2016:MSOP8-0.65-3X3MM, symbol PMIC-ISL97516IUZ-TK_MSOP8_
Connections:
- wire segments 24 -> 55
Other:
- note added: "Allow powering via USB"

Commit message: layout mostly done
Parts:
- C303: symbol CERAMIC-4.7NF-50V-10%-X7R_0603_ -> CERAMIC-4.7NF-50V-10%-X7R_0603_-RESCUE-serial-charger-RESCUE-serial-charger
Connections:
- net GND: now also C303.1; no longer C303.~ (2)
- net at R306.1: now also C303.2; no longer C303.~ (2)
Other:
- moved on the sheet: C303
Changed lines of the file:
@@
 V_BAT
 $Comp
-L GND #PWR011
+L GND #PWR304
 U 1 1 5A53C159
 P 4150 4700
-F 0 "#PWR011" H 4150 4450 50  0001 C CNN
+F 0 "#PWR304" H 4150 4450 50  0001 C CNN
 F 1 "GND" H 4150 4550 50  0000 C CNN
 F 2 "" H 4150 4700 50  0001 C CNN
@@
 $EndComp
 $Comp
-L GND #PWR012
+L GND #PWR305
 U 1 1 5A53C189
 P 4750 4700
-F 0 "#PWR012" H 4750 4450 50  0001 C CNN
+F 0 "#PWR305" H 4750 4450 50  0001 C CNN
 F 1 "GND" H 4750 4550 50  0000 C CNN
 F 2 "" H 4750 4700 50  0001 C CNN
@@
 $EndComp
 $Comp
-L GND #PWR013
+L GND #PWR309
 U 1 1 5A53C1B2
 P 7250 3600
-F 0 "#PWR013" H 7250 3350 50  0001 C CNN
+F 0 "#PWR309" H 7250 3350 50  0001 C CNN
 F 1 "GND" H 7250 3450 50  0000 C CNN
 F 2 "" H 7250 3600 50  0001 C CNN
@@
 $EndComp
 $Comp
-L GND #PWR014
+L GND #PWR313
 U 1 1 5A53D23C
 P 9250 4700
-F 0 "#PWR014" H 9250 4450 50  0001 C CNN
+F 0 "#PWR313" H 9250 4450 50  0001 C CNN
 F 1 "GND" H 9250 4550 50  0000 C CNN
 F 2 "" H 9250 4700 50  0001 C CNN
@@
 $EndComp
 $Comp
-L CERAMIC-4.7NF-50V-10%-X7R_0603_ C303
+L CERAMIC-4.7NF-50V-10%-X7R_0603_-RESCUE-serial-charger-RESCUE-serial-charger C303
 U 1 1 5A53E941
 P 6950 4500
+AR Path="/5A53E941" Ref="C303"  Part="1"
+AR Path="/58D79291/5A53E941" Ref="C303"  Part="1"
 F 0 "C303" H 6800 4550 45  0000 L BNN
 F 1 "CERAMIC-4.7NF-50V-10%-X7R_0603_" H 6800 4400 45  0001 L BNN
@@
 $EndComp
 $Comp
-L GND #PWR015
+L GND #PWR308
 U 1 1 5A53F05F
 P 6950 4700
-F 0 "#PWR015" H 6950 4450 50  0001 C CNN
+F 0 "#PWR308" H 6950 4450 50  0001 C CNN
 F 1 "GND" H 6950 4550 50  0000 C CNN
 F 2 "" H 6950 4700 50  0001 C CNN
@@
 $EndComp
 $Comp
-L GND #PWR016
+L GND #PWR310
 U 1 1 5A53F814
 P 8350 3550
-F 0 "#PWR016" H 8350 3300 50  0001 C CNN
+F 0 "#PWR310" H 8350 3300 50  0001 C CNN
 F 1 "GND" H 8350 3400 50  0000 C CNN
 F 2 "" H 8350 3550 50  0001 C CNN
@@
 $EndComp
 $Comp
-L GND #PWR017
+L GND #PWR311
 U 1 1 5A54005E
 P 8500 3550
-F 0 "#PWR017" H 8500 3300 50  0001 C CNN
+F 0 "#PWR311" H 8500 3300 50  0001 C CNN
 F 1 "GND" H 8500 3400 50  0000 C CNN
 F 2 "" H 8500 3550 50  0001 C CNN
@@
 $EndComp
 $Comp
-L GND #PWR018
+L GND #PWR312
 U 1 1 5A53FE7C
 P 8650 3550
-F 0 "#PWR018" H 8650 3300 50  0001 C CNN
+F 0 "#PWR312" H 8650 3300 50  0001 C CNN
 F 1 "GND" H 8650 3400 50  0000 C CNN
 F 2 "" H 8650 3550 50  0001 C CNN
@@
 $EndComp
 $Comp
-L GND #PWR019
+L GND #PWR314
 U 1 1 5A5404EC
 P 9500 4700
-F 0 "#PWR019" H 9500 4450 50  0001 C CNN
+F 0 "#PWR314" H 9500 4450 50  0001 C CNN
 F 1 "GND" H 9500 4550 50  0000 C CNN
 F 2 "" H 9500 4700 50  0001 C CNN
@@
 $EndComp
 $Comp
-L GND #PWR020
+L GND #PWR306
 U 1 1 5A540C47
 P 5600 4650
-F 0 "#PWR020" H 5600 4400 50  0001 C CNN
+F 0 "#PWR306" H 5600 4400 50  0001 C CNN
 F 1 "GND" H 5600 4500 50  0000 C CNN
 F 2 "" H 5600 4650 50  0001 C CNN
@@
 $EndComp
 $Comp
-L GND #PWR021
+L GND #PWR303
 U 1 1 5A540FA3
 P 3950 4700
-F 0 "#PWR021" H 3950 4450 50  0001 C CNN
+F 0 "#PWR303" H 3950 4450 50  0001 C CNN
 F 1 "GND" H 3950 4550 50  0000 C CNN
 F 2 "" H 3950 4700 50  0001 C CNN
@@
 $EndComp
 $Comp
-L GND #PWR022
+L GND #PWR302
 U 1 1 5A54174B
 P 3750 4700
-F 0 "#PWR022" H 3750 4450 50  0001 C CNN
+F 0 "#PWR302" H 3750 4450 50  0001 C CNN
 F 1 "GND" H 3750 4550 50  0000 C CNN
 F 2 "" H 3750 4700 50  0001 C CNN
@@
 $EndComp
 $Comp
-L GND #PWR023
+L GND #PWR307
 U 1 1 5A543683
 P 6700 4700
-F 0 "#PWR023" H 6700 4450 50  0001 C CNN
+F 0 "#PWR307" H 6700 4450 50  0001 C CNN
 F 1 "GND" H 6700 4550 50  0000 C CNN
 F 2 "" H 6700 4700 50  0001 C CNN
@@
 Connection ~ 3550 3400
 $Comp
-L GND #PWR024
+L GND #PWR301
 U 1 1 5A546E63
 P 3550 4700
-F 0 "#PWR024" H 3550 4450 50  0001 C CNN
+F 0 "#PWR301" H 3550 4450 50  0001 C CNN
 F 1 "GND" H 3550 4550 50  0000 C CNN
 F 2 "" H 3550 4700 50  0001 C CNN
